Commit message: Fix damping problem

File: models/arx7_left.urdf (robot description, URDF)
Before this commit: robot X7LEFT2, 8 links, 7 joints
Links:
- added link eef_link, mass 0.0
Joints:
- added joint gripper_fixed_joint: type fixed, parent link7, child eef_link, origin xyz=0.145 0.0 0.0 rpy=0 0 0

File: models/arx7_right.urdf (robot description, URDF)
Before this commit: robot X7RIGHT2, 8 links, 7 joints
Links:
- added link eef_link, mass 0.0
Joints:
- added joint gripper_fixed_joint: type fixed, parent link7, child eef_link, origin xyz=0.145 0.0 0.0 rpy=0 0 0

Commit message: Update urdf

File: models/arx7_left.urdf (robot description, URDF)
Before this commit: robot X7LEFT2, 9 links, 8 joints
Links:
- link base_link: mass 0.41722 -> 0.44235; geometry collision mesh filename=package://ultron2r_urdf_b/meshes/base_link.STL; visual mesh filename=package://ultron2r_urdf_b/meshes/base_link.STL
- link link1: mass 0.131891884746085 -> 0.0856404273280073; geometry collision mesh filename=package://ultron2r_urdf_b/meshes/link1.STL; visual mesh filename=package://ultron2r_urdf_b/meshes/link1.STL
- link link2: mass 0.971762138327377 -> 1.02244282986255; geometry collision mesh filename=package://ultron2r_urdf_b/meshes/link2.STL; visual mesh filename=package://ultron2r_urdf_b/meshes/link2.STL
- link link3: mass 0.868202345580011 -> 0.80997444672276; geometry collision mesh filename=package://ultron2r_urdf_b/meshes/link3.STL; visual mesh filename=package://ultron2r_urdf_b/meshes/link3.STL
- link link4: mass 0.483750765199191 -> 0.43261626892148; geometry collision mesh filename=package://ultron2r_urdf_b/meshes/link4.STL; visual mesh filename=package://ultron2r_urdf_b/meshes/link4.STL
- link link5: mass 0.59058 -> 0.55065804059678; geometry collision mesh filename=package://ultron2r_urdf_b/meshes/link5.STL; visual mesh filename=package://ultron2r_urdf_b/meshes/link5.STL
- link link6: mass 0.33468 -> 0.369535658973004; geometry collision mesh filename=package://ultron2r_urdf_b/meshes/link6.STL; visual mesh filename=package://ultron2r_urdf_b/meshes/link6.STL
- link link7: mass 0.60047 -> 0.66; geometry collision mesh filename=package://ultron2r_urdf_b/meshes/link7.STL; visual mesh filename=package://ultron2r_urdf_b/meshes/link7.STL
Joints:
- joint joint1: limit lower=-10 upper=10 effort=100 velocity=1000 -> lower=-2.09439 upper=2.09439 effort=100 velocity=1000; origin xyz=0 0.05325 0 rpy=0 0 0 -> xyz=0 -0.0605 0 rpy=3.1416 0 0
- joint joint2: limit lower=-10 upper=10 effort=100 velocity=1000 -> lower=-0 upper=1.5708 effort=100 velocity=1000; origin xyz=0.02725 0.063 0 rpy=0 0 3.1416 -> xyz=0.03125 0.059 0 rpy=-3.1416 0 3.1416
- joint joint3: limit lower=-10 upper=10 effort=100 velocity=1000 -> lower=-0 upper=1.5708 effort=100 velocity=1000; origin xyz=0.02725 0 -0.0865 rpy=-3.1416 0 -3.1416 -> xyz=0.03125 0 -0.0905 rpy=-3.1416 0 3.1416
- joint joint4: limit lower=-10 upper=10 effort=100 velocity=1000 -> lower=-0.17453 upper=1.5708 effort=100 velocity=1000; origin xyz=0 0.02725 0.2165 rpy=0 0 0 -> xyz=0 -0.03125 0.2125 rpy=3.1416 0 0
- joint joint5: limit lower=-10 upper=10 effort=100 velocity=1000 -> lower=-1.5708 upper=1.22173 effort=100 velocity=1000; origin xyz=0.0935 -0.02725 0 rpy=-3.1416 0 0 -> xyz=0.0935 -0.03125 0 rpy=0 0 0
- joint joint6: limit lower=-10 upper=10 effort=100 velocity=1000 -> lower=-0 upper=0.7854 effort=100 velocity=1000; origin xyz=0.1615 -0.04025 0 rpy=-3.1416 0 0 -> xyz=0.1615 0.04025 0 rpy=0 0 0
- joint joint7: limit lower=-10 upper=10 effort=100 velocity=1000 -> lower=-0.7854 upper=0.7854 effort=100 velocity=1000; origin xyz=0 -0.04025 0.022 rpy=3.1416 0 0 -> xyz=0 -0.04025 -0.022 rpy=0 0 0

File: models/arx7_right.urdf (robot description, URDF)
Before this commit: robot X7RIGHT2, 9 links, 8 joints
Links:
- link base_link: mass 0.41722 -> 0.44235; geometry collision mesh filename=package://ultron2r_urdf_b/meshes/base_link.STL; visual mesh filename=package://ultron2r_urdf_b/meshes/base_link.STL
- link link1: mass 0.131891884746085 -> 0.0856404273280073; geometry collision mesh filename=package://ultron2r_urdf_b/meshes/link1.STL; visual mesh filename=package://ultron2r_urdf_b/meshes/link1.STL
- link link2: mass 0.971762294464618 -> 1.02244282986255; geometry collision mesh filename=package://ultron2r_urdf_b/meshes/link2.STL; visual mesh filename=package://ultron2r_urdf_b/meshes/link2.STL
- link link3: mass 0.86819 -> 0.80997444672276; geometry collision mesh filename=package://ultron2r_urdf_b/meshes/link3.STL; visual mesh filename=package://ultron2r_urdf_b/meshes/link3.STL
- link link4: mass 0.483750765199191 -> 0.43261626892148; geometry collision mesh filename=package://ultron2r_urdf_b/meshes/link4.STL; visual mesh filename=package://ultron2r_urdf_b/meshes/link4.STL
- link link5: mass 0.59058 -> 0.55065804059678; geometry collision mesh filename=package://ultron2r_urdf_b/meshes/link5.STL; visual mesh filename=package://ultron2r_urdf_b/meshes/link5.STL
- link link6: mass 0.33468 -> 0.369535658973004; geometry collision mesh filename=package://ultron2r_urdf_b/meshes/link6.STL; visual mesh filename=package://ultron2r_urdf_b/meshes/link6.STL
- link link7: mass 0.600472510680938 -> 0.66; geometry collision mesh filename=package://ultron2r_urdf_b/meshes/link7.STL; visual mesh filename=package://ultron2r_urdf_b/meshes/link7.STL
Joints:
- joint joint1: limit lower=-10 upper=10 effort=100 velocity=1000 -> lower=-2.09439 upper=2.09439 effort=100 velocity=1000; origin xyz=0 -0.05325 0 rpy=3.1416 0 0 -> xyz=0 -0.0605 0 rpy=3.1416 0 0
- joint joint2: limit lower=-10 upper=10 effort=100 velocity=1000 -> lower=-0 upper=1.5708 effort=100 velocity=1000; origin xyz=0.02725 0.063 0 rpy=-3.1416 0 3.1416 -> xyz=0.03125 0.059 0 rpy=-3.1416 0 3.1416
- joint joint3: limit lower=-10 upper=10 effort=100 velocity=1000 -> lower=-0 upper=1.5708 effort=100 velocity=1000; origin xyz=0.02725 0 -0.0865 rpy=3.1416 0 3.1416 -> xyz=0.03125 0 -0.0905 rpy=-3.1416 0 3.1416
- joint joint4: limit lower=-10 upper=10 effort=100 velocity=1000 -> lower=-0.17453 upper=1.5708 effort=100 velocity=1000; origin xyz=0 -0.02725 0.2165 rpy=-3.1416 0 0 -> xyz=0 -0.03125 0.2125 rpy=3.1416 0 0
- joint joint5: limit lower=-10 upper=10 effort=100 velocity=1000 -> lower=-1.5708 upper=1.22173 effort=100 velocity=1000; origin xyz=0.0935 -0.02725 0 rpy=0 0 0 -> xyz=0.0935 -0.03125 0 rpy=0 0 0
- joint joint6: limit lower=-10 upper=10 effort=100 velocity=1000 -> lower=-0 upper=0.7854 effort=100 velocity=1000
- joint joint7: limit lower=-10 upper=10 effort=100 velocity=1000 -> lower=-0.7854 upper=0.7854 effort=100 velocity=1000

Commit message: Fix left urdf

File: models/arx7_left.urdf (robot description, URDF)
Before this commit: robot ultron2r_urdf_b, 9 links, 8 joints
Links:
- link base_link: geometry collision mesh filename=package://ultron2_urdf_g/meshes/base_link.STL; visual mesh filename=package://ultron2_urdf_g/meshes/base_link.STL
- link link1: mass 0.0856404273280073 -> 0.085583; geometry collision mesh filename=package://ultron2_urdf_g/meshes/link1.STL; visual mesh filename=package://ultron2_urdf_g/meshes/link1.STL
- link link2: mass 1.02244282986255 -> 1.02244259916853; geometry collision mesh filename=package://ultron2_urdf_g/meshes/link2.STL; visual mesh filename=package://ultron2_urdf_g/meshes/link2.STL
- link link3: mass 0.80997444672276 -> 0.84083747270065; geometry collision mesh filename=package://ultron2_urdf_g/meshes/link3.STL; visual mesh filename=package://ultron2_urdf_g/meshes/link3.STL
- link link4: mass 0.43261626892148 -> 0.43314458599201; geometry collision mesh filename=package://ultron2_urdf_g/meshes/link4.STL; visual mesh filename=package://ultron2_urdf_g/meshes/link4.STL
- link link5: mass 0.55065804059678 -> 0.552346497691693; geometry collision mesh filename=package://ultron2_urdf_g/meshes/link5.STL; visual mesh filename=package://ultron2_urdf_g/meshes/link5.STL
- link link6: mass 0.369535658973004 -> 0.369986281234796; geometry collision mesh filename=package://ultron2_urdf_g/meshes/link6.STL; visual mesh filename=package://ultron2_urdf_g/meshes/link6.STL
- link link7: mass 0.66 -> 0.073384; geometry collision mesh filename=package://ultron2_urdf_g/meshes/link7.STL; visual mesh filename=package://ultron2_urdf_g/meshes/link7.STL
Joints:
- joint joint1: limit lower=-2.09439 upper=2.09439 effort=100 velocity=1000 -> lower=-10 upper=10 effort=100 velocity=1000; origin xyz=0 -0.0605 0 rpy=3.1416 0 0 -> xyz=0 0.0605 0 rpy=0 0 0
- joint joint2: limit lower=-0 upper=1.5708 effort=100 velocity=1000 -> lower=-10 upper=10 effort=100 velocity=1000; origin xyz=0.03125 0.059 0 rpy=-3.1416 0 3.1416 -> xyz=0.03125 0.059 0 rpy=0 0 3.1416
- joint joint3: limit lower=-0 upper=1.5708 effort=100 velocity=1000 -> lower=-10 upper=10 effort=100 velocity=1000; origin xyz=0.03125 0 -0.0905 rpy=-3.1416 0 3.1416 -> xyz=0.03125 0 -0.0905 rpy=3.1416 0 3.1416
- joint joint4: limit lower=-0.17453 upper=1.5708 effort=100 velocity=1000 -> lower=-10 upper=10 effort=100 velocity=1000; origin xyz=0 -0.03125 0.2125 rpy=3.1416 0 0 -> xyz=0 0.03125 0.2125 rpy=0 0 0
- joint joint5: limit lower=-1.5708 upper=1.22173 effort=100 velocity=1000 -> lower=-10 upper=10 effort=100 velocity=1000; origin xyz=0.0935 -0.03125 0 rpy=0 0 0 -> xyz=0.0935 -0.03125 0 rpy=3.1416 0 0
- joint joint6: limit lower=-0 upper=0.7854 effort=100 velocity=1000 -> lower=-10 upper=10 effort=100 velocity=1000; origin xyz=0.1615 0.04025 0 rpy=0 0 0 -> xyz=0.1615 -0.03425 0 rpy=-3.1416 0 0
- joint joint7: limit lower=-0.7854 upper=0.7854 effort=100 velocity=1000 -> lower=-10 upper=10 effort=100 velocity=1000; origin xyz=0 -0.04025 -0.022 rpy=0 0 0 -> xyz=0 -0.03425 0.022 rpy=-3.1416 0 0

Commit message: Fix

File: models/arx7_left.urdf (robot description, URDF)
Before this commit: robot ultron2_urdf_g, 9 links, 8 joints
Links:
- link link7: mass 0.073384 -> 0.66
